File: channel_splitter/channel_splitter.kicad_sch (KiCad schematic)
At the start: 62 parts, among them J1 USB_B, J4 Conn_01x05, Q1 MMBT3906, SW1 CUI DS03-254-02BE, U1 ATmega328P-AU, U2 TLP2361, U3 74LS32, U4 74LVC1G125, Y1 CSTNE16M0V530000R0

Commit message: Misc local changes
Parts:
- R1, R16: value 220R -> 1k
Changed lines of the file:
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@@
       (effects (font (size 1.27 1.27)))
     )
-    (property "Value" "220R" (at 382.27 228.6 90)
+    (property "Value" "1k" (at 382.27 228.6 90)
       (effects (font (size 1.27 1.27)))
     )
@@
       (effects (font (size 1.27 1.27)) (justify left))
     )
-    (property "Value" "220R" (at 92.71 236.22 0)
+    (property "Value" "1k" (at 92.71 236.22 0)
       (effects (font (size 1.27 1.27)) (justify left))
     )
